File: OCP-2/OCP-2.sch (KiCad schematic (older format))
At the start: 3 parts

Commit message: обвес питания МК и ETH
Parts:
- added C1, C10, C11, C7, C8: Конденсатор*10мкФ*16В*0805, N_RLC:Конденсатор_SMD_IEC_0805, symbol eo-engine:Конденсатор*10мкФ*16В*0805
- added C12, C2, C3, C4, C5, C6, C9: Конденсатор*0,1мкФ*25В*0603, N_RLC:Конденсатор_SMD_IEC_0603, symbol eo-engine:Конденсатор*0,1мкФ*25В*0603
- added R1, R2: Резистор*10кОм*0603, N_RLC:Резистор_SMD_0603_0,065_Вт_pnp, symbol eo-engine:Резистор*10кОм*0603
- added XP1, XP2: Вилка*PLD*6контактов*2ряда*вертикальная*AVR, N_X:Вилка_PLD6_вертикальная_AB, symbol eo-engine:Вилка*PLD*6контактов*2ряда*вертикальная*AVR
Connections:
- net 3V3: now also DD1.18 (AVCC), DD1.4 (VCC), DD1.6 (VCC), DD2.18 (AVCC), DD2.4 (VCC), DD2.6 (VCC), DD3.15 (Vddtx(3V3)), DD3.19 (Vddrx(3V3)), DD3.20 (Vddpll(3V3)), DD3.25 (Vddosc(3V3)), DD3.28 (Vdd(3V3)), C10.1, C11.1, C12.1, C2.1, C3.1, C4.1, C5.1, C6.1, C7.1, C8.1, C9.1, R1.1, R2.1
- net MOSI.S: now reaches DD2.15 (PB3(MOSI/OC2))
- net MOSI.S: now also XP1.2B
- net MISO.S: now reaches DD2.16 (PB4(MISO))
- net MISO.S: now also XP1.1A
- net SCK.S: now reaches DD2.17 (PB5(SCK))
- net SCK.S: now also XP1.2A
- net GND: now reaches DD2.21 (GND)
- net GND: now also DD1.21 (GND), DD1.3 (GND), DD1.5 (GND), DD2.3 (GND), DD2.5 (GND), DD3.11 (Vssrx(GND)), DD3.18 (Vsstx(GND)), DD3.2 (Vss(GND)), DD3.21 (Vsspll(GND)), DD3.22 (Vssosc(GND)), C1.1, C10.2, C11.2, C12.2, C2.2, C3.2, C4.2, C5.2, C6.2, C7.2, C8.2, C9.2, XP1.3B, XP2.3B
- net RES.S: now reaches DD2.29 (PC6(RESET))
- net RES.S: now also R2.2, XP1.3A
- net MOSI.M: now reaches DD1.15 (PB3(MOSI/OC2))
- net MOSI.M: now also XP2.2B
- net MISO.M: now reaches DD1.16 (PB4(MISO))
- net MISO.M: now also XP2.1A
- net SCK.M: now reaches DD1.17 (PB5(SCK))
- net SCK.M: now also XP2.2A
- net RES.M: now reaches DD1.29 (PC6(RESET))
- net RES.M: now also R1.2, XP2.3A
- net EXR.CAP: now reaches DD3.1 (Vext.cap)
- net EXR.CAP: now also C1.2
- no-connect marks 0 -> 2

Commit message: схема DI и DO + трассировка
Parts:
- added C13, C14, C15, C16, C17, C18, C19, C20, C21, C22, C23, C24: Конденсатор*0,1мкФ*25В*0603, N_RLC:Конденсатор_SMD_IEC_0603, symbol eo-engine:Конденсатор*0,1мкФ*25В*0603
- added R10, R12, R18, R19, R20, R21, R22, R24, R26, R28, R30, R32, R38, R39, R4, R40, R41, R42, R43, R44, R45, R46, R47, R48, R49, R50, R51, R52, R53, R54, R6, R8: Резистор*1кОм*0603, N_RLC:Резистор_SMD_0603_0,065_Вт_pnp, symbol eo-engine:Резистор*1кОм*0603
- added R11, R13, R14, R15, R16, R17, R23, R25, R27, R29, R3, R31, R33, R34, R35, R36, R37, R5, R7, R9: Резистор*10кОм*0603, N_RLC:Резистор_SMD_0603_0,065_Вт_pnp, symbol eo-engine:Резистор*10кОм*0603
- added VD1, VD10, VD11, VD12, VD13, VD14, VD15, VD16, VD17, VD18, VD19, VD2, VD20, VD3, VD4, VD5, VD6, VD7, VD8, VD9: Стабилитрон*7,5В*SOD80, N_VD_HL:SOD-80, symbol eo-engine:Стабилитрон*7,5В*SOD80
- added VD21, VD22, VD23, VD24, VD25, VD26, VD27, VD28, VD29, VD30, VD31, VD32: Стабилитрон*3,9В*SOD80, N_VD_HL:SOD-80, symbol eo-engine:Стабилитрон*3,9В*SOD80
- added VT1, VT11, VT12, VT13, VT14, VT15, VT2, VT3, VT4, VT5: Транзистор*pnp*0,5А*45В*SOT23, MOTOR_VD_VT_HL:Корпус_КТ-46, symbol eo-engine:Транзистор*pnp*0,5А*45В*SOT23
- added VT10, VT16, VT17, VT18, VT19, VT20, VT6, VT7, VT8, VT9: Транзистор*npn*0,5А*45В*SOT23, MOTOR_VD_VT_HL:Корпус_КТ-46, symbol eo-engine:Транзистор*npn*0,5А*45В*SOT23
Connections:
- net GND: now also C13.1, C14.1, C15.1, C16.1, C17.1, C18.1, C19.1, C20.1, C21.1, C22.1, C23.1, C24.1, R13.2, R14.2, R15.2, R16.2, R17.2, R33.2, R34.2, R35.2, R36.2, R37.2, VD1.1, VD10.1, VD11.1, VD12.1, VD13.1, VD14.1, VD15.1, VD16.1, VD17.1, VD18.1, VD19.1, VD2.1, VD20.1, VD21.1, VD22.1, VD23.1, VD24.1, VD25.1, VD26.1, VD27.1, VD28.1, VD29.1, VD3.1, VD30.1, VD31.1, VD32.1, VD4.1, VD5.1, VD6.1, VD7.1, VD8.1, VD9.1, VT10.2, VT16.2, VT17.2, VT18.2, VT19.2, VT20.2, VT6.2, VT7.2, VT8.2, VT9.2
- new net: R13.1, R4.2, VT6.1
- new net: R18.2, R3.2, VT1.1
- new net: R14.1, R6.2, VT7.1
- new net: R19.2, R5.2, VT2.1
- new net: R15.1, R8.2, VT8.1
- new net: R20.2, R7.2, VT3.1
- new net: R10.2, R16.1, VT9.1
- new net: R21.2, R9.2, VT4.1
- new net: R12.2, R17.1, VT10.1
- new net: R11.2, R22.2, VT5.1
- new net: R24.2, R33.1, VT16.1
- new net: R23.2, R38.2, VT11.1
- new net: R26.2, R34.1, VT17.1
- new net: R25.2, R39.2, VT12.1
- new net: R28.2, R35.1, VT18.1
- new net: R27.2, R40.2, VT13.1
- new net: R30.2, R36.1, VT19.1
- new net: R29.2, R41.2, VT14.1
- new net: R32.2, R37.1, VT20.1
- new net: R31.2, R42.2, VT15.1
- new net 5V: R11.1, R23.1, R25.1, R27.1, R29.1, R3.1, R31.1, R5.1, R7.1, R9.1, VT1.2, VT11.2, VT12.2, VT13.2, VT14.2, VT15.2, VT2.2, VT3.2, VT4.2, VT5.2
- new net DIN1: R43.2
- new net DIN10: R52.2
- new net DIN11: R53.2
- new net DIN12: R54.2
- new net DIN2: R44.2
- new net DIN3: R45.2
- new net DIN4: R46.2
- new net DIN5: R47.2
- new net DIN6: R48.2
- new net DIN7: R49.2
- new net DIN8: R50.2
- new net DIN9: R51.2
- new net DOU10.PNP: VD20.2, VT15.3
- new net DOU5.PNP: VD10.2, VT5.3
- new net DOUT1.NPN: R18.1, VD1.2, VT6.3
- new net DOUT1.PNP: VD6.2, VT1.3
- new net DOUT10.NPN: R42.1, VD15.2, VT20.3
- new net DOUT2.NPN: R19.1, VD2.2, VT7.3
- new net DOUT2.PNP: VD7.2, VT2.3
- new net DOUT3.NPN: R20.1, VD3.2, VT8.3
- new net DOUT3.PNP: VD8.2, VT3.3
- new net DOUT4.NPN: R21.1, VD4.2, VT9.3
- new net DOUT4.PNP: VD9.2, VT4.3
- new net DOUT5.NPN: R22.1, VD5.2, VT10.3
- new net DOUT6.NPN: R38.1, VD11.2, VT16.3
- new net DOUT6.PNP: VD16.2, VT11.3
- new net DOUT7.NPN: R39.1, VD12.2, VT17.3
- new net DOUT7.PNP: VD17.2, VT12.3
- new net DOUT8.NPN: R40.1, VD13.2, VT18.3
- new net DOUT8.PNP: VD18.2, VT13.3
- new net DOUT9.NPN: R41.1, VD14.2, VT19.3
- new net DOUT9.PNP: VD19.2, VT14.3
- new net MC.DIN1: C13.2, R43.1, VD21.2
- new net MC.DIN10: C22.2, R52.1, VD30.2
- new net MC.DIN11: C23.2, R53.1, VD31.2
- new net MC.DIN12: C24.2, R54.1, VD32.2
- new net MC.DIN2: C14.2, R44.1, VD22.2
- new net MC.DIN3: C15.2, R45.1, VD23.2
- new net MC.DIN4: C16.2, R46.1, VD24.2
- new net MC.DIN5: C17.2, R47.1, VD25.2
- new net MC.DIN6: C18.2, R48.1, VD26.2
- new net MC.DIN7: C19.2, R49.1, VD27.2
- new net MC.DIN8: C20.2, R50.1, VD28.2
- new net MC.DIN9: C21.2, R51.1, VD29.2
- new net MC.OUT1: R4.1
- new net MC.OUT10: R32.1
- new net MC.OUT2: R6.1
- new net MC.OUT3: R8.1
- new net MC.OUT4: R10.1
- new net MC.OUT5: R12.1
- new net MC.OUT6: R24.1
- new net MC.OUT7: R26.1
- new net MC.OUT8: R28.1
- new net MC.OUT9: R30.1

Commit message: размещена угловая розетка модуля
Parts:
- added X1, X2: ico*отверстие*М3, N_X:Отверстие_М3, symbol eo-engine:ico*отверстие*М3
- added XP3: Вилка*DIN41612R*64контакта*2ряда*угловая, MOTOR_X:Вилка_СНП306-64ВП21-24-1, symbol eo-engine:Вилка*DIN41612R*64контакта*2ряда*угловая
- added XS1: Розетка*DIN41612R*64контакта*2ряда*угловая, MOTOR_X:Розетка_СНП306-64РП21_угловая, symbol eo-engine:Розетка*DIN41612R*64контакта*2ряда*угловая
Changed lines of the file:
@@
 Text Label 46750 18000 2    138  ~ 0
 DIN12
+$Comp
+L eo-engine:ico*отверстие*М3 X1
+U 1 1 61A064CA
+P 19000 2000
+F 0 "X1" H 18925 2125 50  0001 C CNN
+F 1 "ico*отверстие*М3" H 18975 1875 50  0001 C CNN
+F 2 "N_X:Отверстие_М3" H 18925 2225 50  0001 C CNN
+F 3 "" H 19000 2000 50  0001 C CNN
+	1    19000 2000
+	1    0    0    -1
+$EndComp
+$Comp
+L eo-engine:ico*отверстие*М3 X2
+U 1 1 61A0A2A3
+P 19000 2500
+F 0 "X2" H 18925 2625 50  0001 C CNN
+F 1 "ico*отверстие*М3" H 18975 2375 50  0001 C CNN
+F 2 "N_X:Отверстие_М3" H 18925 2725 50  0001 C CNN
+F 3 "" H 19000 2500 50  0001 C CNN
+	1    19000 2500
+	1    0    0    -1
+$EndComp
 Wire Bus Line
 	29250 1000 29250 21000
@@
 Wire Bus Line
 	11250 8000 11250 20000
+$Comp
+L eo-engine:Вилка*DIN41612R*64контакта*2ряда*угловая XP3
+U 1 1 61A792DC
+P 50500 2500
+F 0 "XP3" H 51250 2800 138 0000 L CNN
+F 1 "Вилка*DIN41612R*64контакта*2ряда*угловая" H 50500 3000 50  0001 C CNN
+F 2 "MOTOR_X:Вилка_СНП306-64ВП21-24-1" H 50500 3200 50  0001 C CNN
+F 3 "" H 52000 2500 50  0001 C CNN
+F 4 "DIN41612R" H 50700 -7100 138 0000 L CNN "INFO"
+F 5 "https://www.chipdip.ru/product/din41612r-ds1118-64m-r23" H 50500 3100 50  0001 C CNN "LINK"
+	1    50500 2500
+	1    0    0    -1
+$EndComp
+$Comp
+L eo-engine:Розетка*DIN41612R*64контакта*2ряда*угловая XS1
+U 1 1 61AA1FC2
+P 54000 2500
+F 0 "XS1" H 54800 2800 138 0000 L CNN
+F 1 "Розетка*DIN41612R*64контакта*2ряда*угловая" H 54000 3000 50  0001 C CNN
+F 2 "MOTOR_X:Розетка_СНП306-64РП21_угловая" H 54000 3200 50  0001 C CNN
+F 3 "" H 54000 2500 50  0001 C CNN
+F 4 "DIN41612R" H 54250 -7100 138 0000 L CNN "INFO"
+F 5 "https://www.chipdip.ru/product/din41612r-ds1118-64f-r23" H 54000 3100 50  0001 C CNN "LINK"
+	1    54000 2500
+	1    0    0    -1
+$EndComp
 $EndSCHEMATC

Commit message: размещена схема DI, схема не подбита
Connections:
- net labels added: DOUT10.PNP, DOUT5.PNP, RESERVE1, RESERVE10, RESERVE11, RESERVE12, RESERVE2, RESERVE3, RESERVE4, RESERVE5, RESERVE6, RESERVE7, RESERVE8, RESERVE9
- net labels removed: DOU10.PNP, DOU5.PNP
- wire segments 453 -> 569
Other:
- moved on the sheet: XS1

Commit message: изменена вилка программирования, вынесена розетка ETH
Parts:
- removed XP2: Вилка*PLD*6контактов*2ряда*вертикальная*AVR, N_X:Вилка_PLD6_вертикальная_AB, symbol eo-engine:Вилка*PLD*6контактов*2ряда*вертикальная*AVR
- added XP2: Вилка*PLD*8контактов*2ряда*вертикальная*AVR+UART, N_X:Вилка_PLD8_вертикальная_AB, symbol eo-engine:Вилка*PLD*8контактов*2ряда*вертикальная*AVR+UART
- added XS2: Розетка*ETH+трансформатор*8p8c, N_X:Розетка_ETH_KLS12-TL002, symbol eo-engine:Розетка*ETH+трансформатор*8p8c
Connections:
- net labels added: RX, TX
- wire segments 569 -> 575
Changed lines of the file:
@@
 MOSI.M
 $Comp
-L eo-engine:Вилка*PLD*6контактов*2ряда*вертикальная*AVR XP2
-U 1 1 6197BBCB
-P 6250 8000
-F 0 "XP2" H 7150 8300 138 0000 L CNN
-F 1 "Вилка*PLD*6контактов*2ряда*вертикальная*AVR" H 6250 8500 50  0001 C CNN
-F 2 "N_X:Вилка_PLD6_вертикальная_AB" H 6250 8700 50  0001 C CNN
-F 3 "" H 6250 8000 50  0001 C CNN
-F 4 "PLD6" H 6750 7100 138 0000 L CNN "INFO"
-F 5 "https://www.chipdip.ru/product/pld-6" H 6250 8600 50  0001 C CNN "LINK"
-	1    6250 8000
-	1    0    0    -1
-$EndComp
-$Comp
 L eo-engine:#метка-GND #GND2
 U 1 1 6197CC43
-P 8000 8750
-F 0 "#GND2" H 8000 8800 50  0001 C CNN
-F 1 "#метка-GND" H 8050 8900 50  0001 C CNN
-F 2 "" H 8000 8750 50  0001 C CNN
-F 3 "" H 8000 8750 50  0001 C CNN
-	1    8000 8750
+P 8750 8625
+F 0 "#GND2" H 8750 8675 50  0001 C CNN
+F 1 "#метка-GND" H 8800 8775 50  0001 C CNN
+F 2 "" H 8750 8625 50  0001 C CNN
+F 3 "" H 8750 8625 50  0001 C CNN
+	1    8750 8625
 	1    0    0    -1
 $EndComp
 Wire Wire Line
-	7750 8600 8000 8600
-Wire Wire Line
-	8000 8600 8000 8750
+	8750 8600 8750 8625
 NoConn ~ 16500 10900
 NoConn ~ 9000 10900
@@
 	50500 8200 49100 8200
 Wire Wire Line
-	50500 8500 49100 8500
+	50500 10300 49100 10300
 Wire Wire Line
-	50500 8800 49100 8800
+	50500 10600 49100 10600
 Wire Wire Line
-	50500 9100 49100 9100
+	50500 10900 49100 10900
 Wire Wire Line
-	50500 9400 49100 9400
+	50500 11200 49100 11200
 Wire Wire Line
-	50500 9700 49100 9700
+	50500 11500 49100 11500
 Wire Wire Line
-	50500 10000 49100 10000
+	50500 11800 49100 11800
 Wire Wire Line
-	50500 10300 49100 10300
+	50500 8500 49100 8500
 Wire Wire Line
-	50500 10600 49100 10600
+	50500 8800 49100 8800
 Wire Wire Line
-	50500 10900 49100 10900
+	50500 9100 49100 9100
 Wire Wire Line
-	50500 11200 49100 11200
+	50500 9400 49100 9400
 $Comp
 L eo-engine:#метка-5V #5V12
@@
 Wire Wire Line
 	52750 2800 52000 2800
-Text Label 49250 8500 0    138  ~ 0
+Text Label 49250 10300 0    138  ~ 0
 DIN1
-Text Label 49250 8800 0    138  ~ 0
+Text Label 49250 10600 0    138  ~ 0
 DIN2
-Text Label 49250 9100 0    138  ~ 0
+Text Label 49250 10900 0    138  ~ 0
 DIN3
-Text Label 49250 9400 0    138  ~ 0
+Text Label 49250 11200 0    138  ~ 0
 DIN4
-Text Label 49250 9700 0    138  ~ 0
+Text Label 49250 11500 0    138  ~ 0
 DIN5
-Text Label 49250 10000 0    138  ~ 0
+Text Label 49250 11800 0    138  ~ 0
 DIN6
-Text Label 49250 10300 0    138  ~ 0
+Text Label 49250 8500 0    138  ~ 0
 DIN7
-Text Label 49250 10600 0    138  ~ 0
+Text Label 49250 8800 0    138  ~ 0
 DIN8
-Text Label 49250 10900 0    138  ~ 0
+Text Label 49250 9100 0    138  ~ 0
 DIN9
 Wire Wire Line
-	50500 11500 49100 11500
+	50500 9700 49100 9700
 Wire Wire Line
-	50500 11800 49100 11800
-Text Label 49250 11200 0    138  ~ 0
+	50500 10000 49100 10000
+Text Label 49250 9400 0    138  ~ 0
 DIN10
-Text Label 49250 11500 0    138  ~ 0
+Text Label 49250 9700 0    138  ~ 0
 DIN11
-Text Label 49250 11800 0    138  ~ 0
+Text Label 49250 10000 0    138  ~ 0
 DIN12
 Wire Wire Line
@@
 	59500 8200 60900 8200
 Wire Wire Line
-	59500 8500 60900 8500
+	59500 10300 60900 10300
 Wire Wire Line
-	59500 8800 60900 8800
+	59500 10600 60900 10600
 Wire Wire Line
-	59500 9100 60900 9100
+	59500 10900 60900 10900
 Wire Wire Line
-	59500 9400 60900 9400
+	59500 11200 60900 11200
 Wire Wire Line
-	59500 9700 60900 9700
+	59500 11500 60900 11500
 Wire Wire Line
-	59500 10000 60900 10000
+	59500 11800 60900 11800
 Wire Wire Line
-	59500 10300 60900 10300
+	59500 8500 60900 8500
 Wire Wire Line
-	59500 10600 60900 10600
+	59500 8800 60900 8800
 Wire Wire Line
-	59500 10900 60900 10900
+	59500 9100 60900 9100
 Wire Wire Line
-	59500 11200 60900 11200
-Text Label 60750 8500 2    138  ~ 0
+	59500 9400 60900 9400
+Text Label 60750 10300 2    138  ~ 0
 DIN1
-Text Label 60750 8800 2    138  ~ 0
+Text Label 60750 10600 2    138  ~ 0
 DIN2
-Text Label 60750 9100 2    138  ~ 0
+Text Label 60750 10900 2    138  ~ 0
 DIN3
-Text Label 60750 9400 2    138  ~ 0
+Text Label 60750 11200 2    138  ~ 0
 DIN4
-Text Label 60750 9700 2    138  ~ 0
+Text Label 60750 11500 2    138  ~ 0
 DIN5
-Text Label 60750 10000 2    138  ~ 0
+Text Label 60750 11800 2    138  ~ 0
 DIN6
-Text Label 60750 10300 2    138  ~ 0
+Text Label 60750 8500 2    138  ~ 0
 DIN7
-Text Label 60750 10600 2    138  ~ 0
+Text Label 60750 8800 2    138  ~ 0
 DIN8
-Text Label 60750 10900 2    138  ~ 0
+Text Label 60750 9100 2    138  ~ 0
 DIN9
 Wire Wire Line
-	59500 11500 60900 11500
+	59500 9700 60900 9700
 Wire Wire Line
-	59500 11800 60900 11800
-Text Label 60750 11200 2    138  ~ 0
+	59500 10000 60900 10000
+Text Label 60750 9400 2    138  ~ 0
 DIN10
-Text Label 60750 11500 2    138  ~ 0
+Text Label 60750 9700 2    138  ~ 0
 DIN11
-Text Label 60750 11800 2    138  ~ 0
+Text Label 60750 10000 2    138  ~ 0
 DIN12
+$Comp
+L eo-engine:Вилка*PLD*8контактов*2ряда*вертикальная*AVR+UART XP2
+U 1 1 61ACE107
+P 6250 8000
+F 0 "XP2" H 7125 8275 138 0000 L CNN
+F 1 "Вилка*PLD*8контактов*2ряда*вертикальная*AVR+UART" H 6250 8500 50  0001 C CNN
+F 2 "N_X:Вилка_PLD8_вертикальная_AB" H 6250 8700 50  0001 C CNN
+F 3 "" H 6250 8000 50  0001 C CNN
+F 4 "PLD8" H 6750 6825 138 0000 L CNN "INFO"
+F 5 "https://www.chipdip.ru/product/pld-8-ds1021-2x4" H 6250 8600 50  0001 C CNN "LINK"
+	1    6250 8000
+	1    0    0    -1
+$EndComp
+Wire Wire Line
+	7750 8600 8750 8600
+Text Label 10000 13900 2    138  ~ 0
+RX
+Wire Wire Line
+	9000 13900 10150 13900
+Entry Wire Line
+	10150 13900 10250 14000
+Text Label 10000 14200 2    138  ~ 0
+TX
+Wire Wire Line
+	9000 14200 10150 14200
+Entry Wire Line
+	10250 14100 10150 14200
+Text Label 4000 8900 0    138  ~ 0
+RX
+Text Label 10000 9250 2    138  ~ 0
+TX
+Wire Wire Line
+	3850 8900 6250 8900
+Entry Wire Line
+	3750 9000 3850 8900
+Entry Wire Line
+	10250 9350 10150 9250
+Wire Wire Line
+	7750 8900 8250 8900
+Wire Wire Line
+	8250 8900 8250 9250
+Wire Wire Line
+	8250 9250 10150 9250
 Wire Bus Line
 	29250 1000 29250 21000
@@
 	17750 8000 17750 20000
 Wire Bus Line
-	10250 8000 10250 20000
-Wire Bus Line
 	18750 9500 18750 20000
 Wire Bus Line
@@
 Wire Bus Line
 	11250 8000 11250 20000
+Wire Bus Line
+	10250 8000 10250 20000
+$Comp
+L eo-engine:Розетка*ETH+трансформатор*8p8c XS2
+U 1 1 61F755EC
+P 5000 2500
+F 0 "XS2" H 5625 2800 138 0000 R CNN
+F 1 "Розетка*ETH+трансформатор*8p8c" H 5000 3000 50  0001 C CNN
+F 2 "N_X:Розетка_ETH_KLS12-TL002" H 5000 3200 50  0001 C CNN
+F 3 "" H 5000 2500 50  0001 C CNN
+F 4 "RJ45" H 6425 -1075 138 0000 R CNN "INFO"
+F 5 "https://www.chipdip.ru/product/sk02-111015nl" H 5000 3100 50  0001 C CNN "LINK"
+	1    5000 2500
+	-1   0    0    -1
+$EndComp
 $EndSCHEMATC

Commit message: схема подключения ETH без SPI и светодиодов
Parts:
- added C25, C26: Конденсатор*10мкФ*16В*0805, N_RLC:Конденсатор_SMD_IEC_0805, symbol eo-engine:Конденсатор*10мкФ*16В*0805
- added C27, C28: Конденсатор*12пФ*50В*0603, N_RLC:Конденсатор_SMD_IEC_0603, symbol eo-engine:Конденсатор*12пФ*50В*0603
- added C29, C30: Конденсатор*0,1мкФ*25В*0603, N_RLC:Конденсатор_SMD_IEC_0603, symbol eo-engine:Конденсатор*0,1мкФ*25В*0603
- added G1: LDO*вход_18Вmax*выход_3,3В*ток_1,2АSOT-223, N_VD_HL:Транзистор_NPN_SOT223_pnp, symbol eo-engine:LDO*вход_18Вmax*выход_3,3В*ток_1,2АSOT-223
- added L1: Чип-индуктивность*0,56мкГн*150мА*0805, N_RLC:Резистор_SMD_IEC_0805_0,125_Вт, symbol eo-engine:Чип-индуктивность*0,56мкГн*150мА*0805
- added R55, R56, R57, R58: Резистор*49,9кОм*0603, N_RLC:Резистор_SMD_0603_0,065_Вт_pnp, symbol eo-engine:Резистор*49,9Ом*0603
- added R59: Резистор*2,32кОм*0603, N_RLC:Резистор_SMD_0603_0,065_Вт_pnp, symbol eo-engine:Резистор*2,32кОм*0603
- added ZQ1: Резонатор*25МГц*HC-49U, N_RLC:Резонатор_РК456МДУ(DIP), symbol eo-engine:Резонатор*25МГц*HC-49U
Connections:
- net labels added: MID-TX, OSC1, OSC2, RBIAS, TPIN+, TPIN-, TPOUT+, TPOUT-
- wire segments 575 -> 638
- no-connect marks 2 -> 3
Other:
- note added: "подключить светодиоды, подключить SPI"
- moved on the sheet: C1, C10, C11, C12, C2, C3, C4, C5, C6, C7, C8, C9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

Commit message: полная схема подключен ETH и МК, нет клеммников
Parts:
- added R60, R61, R64, R65: Резистор*1кОм*0603, N_RLC:Резистор_SMD_0603_0,065_Вт_pnp, symbol eo-engine:Резистор*1кОм*0603
- added R62, R63: Резистор*10кОм*0603, N_RLC:Резистор_SMD_0603_0,065_Вт_pnp, symbol eo-engine:Резистор*10кОм*0603
Connections:
- net labels added: ETH.CLK, ETH.CS, ETH.INT, ETH.MISO, ETH.MOSI, ETH.RES, LEDA, LEDB, SCL, SDA
- wire segments 638 -> 702
- no-connect marks 3 -> 13
Other:
- note added: "MASTER"
- note added: "SLAVE"
- note added: "подключить SPI"
- note removed: "подключить светодиоды, подключить SPI"
- moved on the sheet: C10, C11, C12, C25, C26, C29, C30, C7, C8, C9, DD1, DD2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

Commit message: схема включения ETH + клеммники вместо СНП306
Parts:
- removed XP3: Вилка*DIN41612R*64контакта*2ряда*угловая, MOTOR_X:Вилка_СНП306-64ВП21-24-1, symbol eo-engine:Вилка*DIN41612R*64контакта*2ряда*угловая
- removed XS1: Розетка*DIN41612R*64контакта*2ряда*угловая, MOTOR_X:Розетка_СНП306-64РП21_угловая, symbol eo-engine:Розетка*DIN41612R*64контакта*2ряда*угловая
- added X3, X4: ico*отверстие*М3, N_X:Отверстие_М3, symbol eo-engine:ico*отверстие*М3
- added XP10, XP11, XP12, XP13, XP4, XP5, XP6, XP7, XP8, XP9: Вилка*PLS*3контактов*1ряд*вертикальная, N_X:Вилка_PLS3_вертикальная, symbol eo-engine:Вилка*PLS*3контактов*1ряд*вертикальная
- added XP14, XP15, XP16, XP17, XP18: Клеммник*шаг_3,5*5контактов*1ряд*вертикальная, N_X:Клеммник_15EDGVC-3.5-05P, symbol eo-engine:Клеммник*шаг_3,5*5контактов*1ряд*вертикальная
- added XP19: Клеммник*шаг_3,5*3контактов*1ряд*вертикальная, N_X:Клеммник_15EDGVC-3.5-03P, symbol eo-engine:Клеммник*шаг_3,5*3контактов*1ряд*вертикальная
Connections:
- net labels added: DOUT1, DOUT10, DOUT2, DOUT3, DOUT4, DOUT5, DOUT6, DOUT7, DOUT8, DOUT9
- net labels removed: RESERVE1, RESERVE10, RESERVE11, RESERVE12, RESERVE2, RESERVE3, RESERVE4, RESERVE5, RESERVE6, RESERVE7, RESERVE8, RESERVE9
- wire segments 702 -> 654
- no-connect marks 13 -> 16
Other:
- note removed: "10 входов\n10 выходов\nETH"
